File: CONTROL.kicad_sch (KiCad schematic)
At the start: 8 parts, among them U10 ATF22V10C, U11 ATF22V10C, U8 ATF22V10C, U9 ATF22V10C

Commit message: V1C version of BITSY that uses an SRAM SIMM for memory.
This version sent to JLCPCB on 08/15/2025.
Connections:
- net ~{RAM1CS}: now reaches U9.20 (IO3)
- net ~{RAMCS} renamed ~{RAM0CS}
- net ~{RDEVEN}: no longer names the net of U11.20 (IO3)
- net ~{RDODD} renamed ~{READ}
Changed lines of the file:
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@@
 	(title_block
 		(title "BITSY Mark I - An MC68000 Single Board Computer")
-		(date "2025-06-12")
-		(rev "V1B")
+		(date "2025-08-15")
+		(rev "V1C")
 		(comment 1 "Licensed under CC-BY-SA-NC 4.0.")
 		(comment 2 "https://github.com/codesmythe/BITSY_MK_I")
@@
 	)
 	(no_connect
+		(at 158.75 111.76)
+	)
+	(no_connect
 		(at 212.09 109.22)
 	)
@@
 	)
 	(no_connect
-		(at 68.58 106.68)
-	)
-	(no_connect
 		(at 252.73 119.38)
 	)
@@
 	(wire
 		(pts
+			(xy 68.58 106.68) (xy 83.82 106.68)
+		)
+		(stroke
+			(width 0)
+			(type default)
+		)
+	)
+	(wire
+		(pts
 			(xy 256.54 109.22) (xy 242.57 109.22)
 		)
@@
 	(wire
 		(pts
-			(xy 158.75 111.76) (xy 168.91 111.76)
-		)
-		(stroke
-			(width 0)
-			(type default)
-		)
-	)
-	(wire
-		(pts
 			(xy 256.54 81.28) (xy 256.54 104.14)
 		)
@@
 		)
 	)
-	(label "~{RDEVEN}"
-		(at 161.29 111.76 0)
-		(effects
-			(font
-				(size 1.27 1.27)
-			)
-			(justify left bottom)
-		)
-	)
 	(label "R~{W}"
 		(at 242.57 129.54 0)
@@
 		)
 	)
-	(label "~{RAMCS}"
+	(label "~{RAM0CS}"
 		(at 72.39 111.76 0)
 		(effects
@@
 		)
 	)
+	(label "~{RAM1CS}"
+		(at 72.39 106.68 0)
+		(effects
+			(font
+				(size 1.27 1.27)
+			)
+			(justify left bottom)
+		)
+	)
 	(label "R~{W}"
 		(at 161.29 121.92 0)
@@
 		)
 	)
-	(label "~{RDODD}"
+	(label "~{READ}"
 		(at 161.29 114.3 0)
 		(effects
@@
 		)
 	)
-	(hierarchical_label "~{RAMCS}"
+	(hierarchical_label "~{RAM0CS}"
 		(shape output)
 		(at 83.82 111.76 0)
@@
 		)
 	)
-	(hierarchical_label "~{RDODD}"
+	(hierarchical_label "~{READ}"
 		(shape output)
 		(at 168.91 114.3 0)
@@
 		)
 	)
-	(hierarchical_label "~{RDEVEN}"
-		(shape output)
-		(at 168.91 111.76 0)
-		(effects
-			(font
-				(size 1.27 1.27)
-			)
-			(justify left)
-		)
-	)
 	(hierarchical_label "~{RESET}"
 		(shape input)
@@
 		(effects
 			(font
+				(size 1.27 1.27)
+			)
+			(justify left)
+		)
+	)
+	(hierarchical_label "~{RAM1CS}"
+		(shape output)
+		(at 83.82 106.68 0)
+		(effects
+			(font

Commit message: Update part numbers.
Parts:
- U10, U11, U8, U9: PartNum01 737-ICS-324-T -> 737-ICM-324-1-GT-HT
Changed lines of the file:
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@@
 			)
 		)
-		(property "PartNum01" "737-ICS-324-T"
+		(property "PartNum01" "737-ICM-324-1-GT-HT"
 			(at 143.51 52.07 0)
 			(effects
@@
 			)
 		)
-		(property "PartNum01" "737-ICS-324-T"
+		(property "PartNum01" "737-ICM-324-1-GT-HT"
 			(at 53.34 110.49 0)
 			(effects
@@
 			)
 		)
-		(property "PartNum01" "737-ICS-324-T"
+		(property "PartNum01" "737-ICM-324-1-GT-HT"
 			(at 227.33 115.57 0)
 			(effects
@@
 			)
 		)
-		(property "PartNum01" "737-ICS-324-T"
+		(property "PartNum01" "737-ICM-324-1-GT-HT"
 			(at 143.51 115.57 0)
 			(effects
