File: IDE.kicad_sch (KiCad schematic)
At the start: 7 parts, among them J4 Conn_02x22_Odd_Even, U14 74HCT245, U15 74HCT245

Commit message: Update part numbers.
Parts:
- U14, U15: PartNum01 737-ICS-320-T -> 737-ICM-320-1-GT-HT
Changed lines of the file:
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@@
 			)
 		)
-		(property "PartNum01" "737-ICS-320-T"
+		(property "PartNum01" "737-ICM-320-1-GT-HT"
 			(at 85.09 36.83 0)
 			(effects
@@
 			)
 		)
-		(property "PartNum01" "737-ICS-320-T"
+		(property "PartNum01" "737-ICM-320-1-GT-HT"
 			(at 85.09 96.52 0)
 			(effects
