File: PWRRESET.kicad_sch (KiCad schematic)
At the start: 9 parts, among them J1 Barrel_Jack_Switch, Q1 2N7000, SW1 RESET_SW, U7 MIC1232

Commit message: Update part numbers.
Parts:
- D1: PartNum00 696-SSL-LX5093GT -> 859-LTL-307GLC
- U7: PartNum01 571-1-2199298-2 -> 737-ICM-308-1-GT-HT
Changed lines of the file:
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@@
 			)
 		)
-		(property "PartNum00" "696-SSL-LX5093GT"
+		(property "PartNum00" "859-LTL-307GLC"
 			(at 100.33 91.44 0)
 			(effects
@@
 			)
 		)
-		(property "PartNum01" "571-1-2199298-2"
-			(at 147.32 99.06 0)
-			(effects
+		(property "PartNum01" "737-ICM-308-1-GT-HT"
+			(at 147.32 99.06 0)
+			(effects
